File: geiger2.sch (EAGLE design)
At the start: 22 parts, among them Q1 IRF740, U1 STM32F042KXTX

Commit message: Finish schematic v1.0
Parts:
- added C10, C11, C12, C13, C14, C15, C16, C8, C9: (no value), rcl:C-EUC0805
- added C17: (no value), rcl:C-EUC1206K
- added C18: (no value), rcl:C-EUC0805K
- added D4: (no value), dp_devices:DIODE-SOD-123
- added IC2: REG1117, burr-brown:REG1117
- added JP1, JP2: (no value), pinhead:PINHD-1X2
- added JP3: (no value), pinhead:PINHD-1X3
- added L2, L3: (no value), dp_devices:FERRITE-0805
- added OK1, OK10, OK11, OK12, OK13, OK14, OK2, OK3, OK4, OK5, OK6, OK7, OK8, OK9: PC817, optocoupler:PC817
- added Q2: CSM-7X-DU, crystal:CSM-7X-DU
- added R10, R11, R12, R13, R14, R15, R16, R17, R18, R19, R20, R22, R25, R26, R27, R28, R29, R30, R31, R32, R33, R34, R7, R8, R9: (no value), rcl:R-EU_R0805
- added R21, R23, R24: (no value), rcl:R-EU_R1206
- added S1, S2, S3: (no value), switch-omron:10-XX
- added SG1: BUZZERSMD2-KIT, SparkFun:BUZZERSMD2-KIT
- added T3: (no value), transistor:BC857A-PNP-SOT23-BEC
- added T4: (no value), transistor:BC847-NPN-SOT23-BEC
- added T5: BC847, transistor-neu-to92:BC847
- added X1: 22-23-2021, con-molex:22-23-2021
- added X2, X4: 22-23-2041, con-molex:22-23-2041
- added X3: 22-23-2101, con-molex:22-23-2101
- R4: device rcl:R-EU_M1206 -> rcl:R-EU_R2512
Connections:
- new net +12V: C14.1, IC2.VIN, L3.2, X1-2.S
- new net +3V3: C10.1, C11.1, C8.1, C9.1, D4.C, L2.2, R22.2, R26.2, R29.2, R32.2, R33.2, R34.1, SG1.2, T3.E, U1.VDD, U1.VDDA, U1.VDDIO2, X2-4.S
- new net N$13: C12.1, U1.NRST
- new net N$14: OK14.A, R20.2
- new net N$15: OK13.A, R19.2
- new net N$16: OK12.A, R18.2
- new net N$17: OK11.A, R17.2
- new net N$18: C1.+, L3.1, R4.2, T2.E, U$1.DRV_COLL, U$1.SW_COLL, U$1.VCC
- new net N$19: OK10.A, R16.2
- new net N$20: OK9.A, R15.2
- new net N$21: OK8.A, R14.2
- new net N$22: OK7.A, R13.2
- new net N$23: OK6.A, R12.2
- new net N$24: OK5.A, R11.2
- new net N$25: OK4.A, R10.2
- new net N$26: OK3.A, R9.2
- new net N$27: OK2.A, R8.2
- new net N$28: OK1.A, R7.2
- new net N$29: OK1.COL, OK2.COL, OK3.COL, OK4.COL, R21.1
- new net N$30: U1.PA13, X2-3.S
- new net N$31: U1.PA14, X2-2.S
- new net N$32: OK2.EMIT, X4-2.S
- new net N$33: OK3.EMIT, X4-3.S
- new net N$34: OK4.EMIT, X4-4.S
- new net N$35: C15.1, Q2.1, U1.PF1-OSC_OUT
- new net N$36: OK5.COL, X3-1.S
- new net N$37: OK6.COL, X3-2.S
- new net N$38: OK5.EMIT
- new net N$39: OK7.COL, X3-3.S
- new net N$40: OK8.COL, X3-4.S
- new net N$41: OK9.COL, X3-5.S
- new net N$42: OK10.COL, X3-6.S
- new net N$43: OK11.COL, X3-7.S
- new net N$44: OK12.COL, X3-8.S
- new net N$45: OK13.COL, X3-9.S
- new net N$46: OK14.COL, X3-10.S
- new net N$47: C16.1, Q2.2, U1.PF0-OSC_IN
- new net N$48: JP1.2, R22.1, U1.PB8-BOOT0
- new net N$49: R23.2, R24.1
- new net N$50: C17.1, JP2.2, R24.2
- new net N$51: R27.2, T3.C
- new net N$52: C17.2, R25.2
- new net N$53: R25.1, R26.1, T3.B
- new net N$54: C18.1, R27.1, R28.1, T4.B
- new net N$55: JP3.3, U1.PA9
- new net N$56: JP3.2, U1.PA10
- new net N$57: R29.1, T4.C, U1.PA15
- new net N$58: R30.2, U1.PA8
- new net N$59: R30.1, R31.2, T5.B
- new net N$60: R33.1, S1.P, S1.P1
- new net N$61: D4.A, SG1.1, T5.E
- new net N$63: R32.1, S2.P, S2.P1
- new net N$64: R34.2, S3.P, S3.P1
- new net OK1: R11.1, U1.PA0
- new net OK10: R20.1, U1.PA12
- new net OK11: R7.1, U1.PB0
- new net OK12: R8.1, U1.PB1
- new net OK13: R9.1, U1.PB3
- new net OK14: R10.1, U1.PB4
- new net OK2: R12.1, U1.PA1
- new net OK3: R13.1, U1.PA2
- new net OK4: R14.1, U1.PA3
- new net OK5: R15.1, U1.PA4
- new net OK6: R16.1, U1.PA5
- new net OK7: R17.1, U1.PA6
- new net OK8: R18.1, U1.PA7
- new net OK9: R19.1, U1.PA11
- new net V+: C3.+, D1.C, D2.A, R21.2
- net GND: now also C10.2, C11.2, C12.2, C13.2, C14.2, C15.2, C16.2, C18.2, C8.2, C9.2, IC2.GND, JP1.1, JP2.1, JP3.1, OK1.C, OK10.C, OK10.EMIT, OK11.C, OK11.EMIT, OK12.C, OK12.EMIT, OK13.C, OK13.EMIT, OK14.C, OK14.EMIT, OK2.C, OK3.C, OK4.C, OK5.C, OK6.C, OK6.EMIT, OK7.C, OK7.EMIT, OK8.C, OK8.EMIT, OK9.C, OK9.EMIT, R28.2, R31.1, S1.S, S1.S1, S2.S, S2.S1, S3.S, S3.S1, T4.E, T5.C, U1.PB5, U1.PB6, U1.PB7, U1.VSS1, U1.VSS2, X1-1.S, X2-1.S
- net N$2: now also R23.1
- net N$8: now also OK1.EMIT, X4-1.S; no longer C3.+, D1.C, D2.A
- net N$9: now also C13.1, IC2.VOUT, L2.1; no longer C1.+, R4.2, T2.E, U$1.DRV_COLL, U$1.SW_COLL, U$1.VCC
Other:
- moved on the sheet: U1

Commit message: Edit schematic
Connections:
- removed net N$61: D4.A, SG1.1, T5.E
- new net N$62: D4.A, SG1.1, T5.C
- net GND: now also T5.E; no longer T5.C
Other:
- moved on the sheet: T5
Changed lines of the file:
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@@
 <setting verticaltext="up"/>
 </settings>
-<grid distance="0.1" unitdist="inch" unit="inch" style="lines" multiple="1" display="yes" altdistance="0.01" altunitdist="inch" altunit="inch"/>
+<grid distance="0.1" unitdist="inch" unit="inch" style="lines" multiple="1" display="no" altdistance="0.01" altunitdist="inch" altunit="inch"/>
 <layers>
 <layer number="1" name="Top" color="4" fill="1" visible="no" active="no"/>
@@
 <attribute name="VALUE" x="198.12" y="55.88" size="1.778" layer="96"/>
 </instance>
-<instance part="T5" gate="G$1" x="162.56" y="83.82" smashed="yes" rot="R180">
-<attribute name="NAME" x="172.72" y="76.2" size="1.778" layer="95" rot="R180"/>
-<attribute name="VALUE" x="172.72" y="78.74" size="1.778" layer="96" rot="R180"/>
+<instance part="T5" gate="G$1" x="162.56" y="83.82" smashed="yes" rot="MR0">
+<attribute name="NAME" x="172.72" y="91.44" size="1.778" layer="95" rot="MR0"/>
+<attribute name="VALUE" x="172.72" y="88.9" size="1.778" layer="96" rot="MR0"/>
 </instance>
 <instance part="SG1" gate="G$1" x="157.48" y="93.98" smashed="yes" rot="R90">
@@
 <pinref part="GND36" gate="1" pin="GND"/>
 <wire x1="177.8" y1="68.58" x2="160.02" y2="68.58" width="0.1524" layer="91"/>
-<pinref part="T5" gate="G$1" pin="C"/>
+<pinref part="T5" gate="G$1" pin="E"/>
 <wire x1="160.02" y1="78.74" x2="160.02" y2="68.58" width="0.1524" layer="91"/>
 <junction x="160.02" y="68.58"/>
@@
 <segment>
 <pinref part="R30" gate="G$1" pin="1"/>
-<pinref part="T5" gate="G$1" pin="B"/>
 <wire x1="187.96" y1="83.82" x2="177.8" y2="83.82" width="0.1524" layer="91"/>
 <pinref part="R31" gate="G$1" pin="2"/>
-<wire x1="177.8" y1="83.82" x2="165.1" y2="83.82" width="0.1524" layer="91"/>
 <wire x1="177.8" y1="81.28" x2="177.8" y2="83.82" width="0.1524" layer="91"/>
+<pinref part="T5" gate="G$1" pin="B"/>
+<wire x1="165.1" y1="83.82" x2="177.8" y2="83.82" width="0.1524" layer="91"/>
 <junction x="177.8" y="83.82"/>
-</segment>
-</net>
-<net name="N$61" class="0">
-<segment>
-<pinref part="T5" gate="G$1" pin="E"/>
-<pinref part="SG1" gate="G$1" pin="1"/>
-<wire x1="160.02" y1="88.9" x2="160.02" y2="93.98" width="0.1524" layer="91"/>
-<pinref part="D4" gate="D" pin="A"/>
-<wire x1="167.64" y1="93.98" x2="167.64" y2="88.9" width="0.1524" layer="91"/>
-<wire x1="167.64" y1="88.9" x2="160.02" y2="88.9" width="0.1524" layer="91"/>
-<junction x="160.02" y="88.9"/>
 </segment>
 </net>
@@
 </segment>
 </net>
+<net name="N$62" class="0">
+<segment>
+<pinref part="T5" gate="G$1" pin="C"/>
+<pinref part="SG1" gate="G$1" pin="1"/>
+<wire x1="160.02" y1="88.9" x2="160.02" y2="93.98" width="0.1524" layer="91"/>
+<pinref part="D4" gate="D" pin="A"/>
+<wire x1="160.02" y1="88.9" x2="167.64" y2="88.9" width="0.1524" layer="91"/>
+<wire x1="167.64" y1="88.9" x2="167.64" y2="93.98" width="0.1524" layer="91"/>
+<junction x="160.02" y="88.9"/>
+</segment>
+</net>

Commit message: Edit mosfet driver
Connections:
- net GND: now also T2.C; no longer T1.C
- net N$18: now also T1.C; no longer T2.E
- net N$6: now also T2.E; no longer T2.C
Other:
- moved on the sheet: T1, T2
Changed lines of the file:
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@@
 <?xml version="1.0" encoding="utf-8"?>
 <!DOCTYPE eagle SYSTEM "eagle.dtd">
-<eagle version="9.3.0">
+<eagle version="9.4.1">
 <drawing>
 <settings>
@@
 <setting verticaltext="up"/>
 </settings>
-<grid distance="0.1" unitdist="inch" unit="inch" style="lines" multiple="1" display="no" altdistance="0.01" altunitdist="inch" altunit="inch"/>
+<grid distance="0.1" unitdist="inch" unit="inch" style="lines" multiple="1" display="yes" altdistance="0.01" altunitdist="inch" altunit="inch"/>
 <layers>
 <layer number="1" name="Top" color="4" fill="1" visible="no" active="no"/>
@@
 <attribute name="VALUE" x="91.694" y="57.531" size="1.778" layer="96"/>
 </instance>
-<instance part="T1" gate="G$1" x="66.04" y="30.48" smashed="yes" rot="MR180">
-<attribute name="NAME" x="60.96" y="27.94" size="1.778" layer="95" rot="MR180"/>
-<attribute name="VALUE" x="55.88" y="25.4" size="1.778" layer="96" rot="MR180"/>
-</instance>
-<instance part="T2" gate="G$1" x="66.04" y="45.72" smashed="yes">
-<attribute name="NAME" x="63.5" y="50.8" size="1.778" layer="95"/>
+<instance part="T1" gate="G$1" x="66.04" y="45.72" smashed="yes">
+<attribute name="NAME" x="60.96" y="48.26" size="1.778" layer="95"/>
 <attribute name="VALUE" x="55.88" y="50.8" size="1.778" layer="96"/>
+</instance>
+<instance part="T2" gate="G$1" x="66.04" y="30.48" smashed="yes">
+<attribute name="NAME" x="63.5" y="35.56" size="1.778" layer="95"/>
+<attribute name="VALUE" x="55.88" y="35.56" size="1.778" layer="96"/>
 </instance>
 <instance part="Q1" gate="G$1" x="83.82" y="40.64" smashed="yes">
@@
 <wire x1="27.94" y1="5.08" x2="17.78" y2="5.08" width="0.1524" layer="91"/>
 <junction x="17.78" y="5.08"/>
-<pinref part="T1" gate="G$1" pin="C"/>
-<wire x1="68.58" y1="25.4" x2="68.58" y2="5.08" width="0.1524" layer="91"/>
-<wire x1="68.58" y1="5.08" x2="43.18" y2="5.08" width="0.1524" layer="91"/>
+<wire x1="86.36" y1="5.08" x2="68.58" y2="5.08" width="0.1524" layer="91"/>
 <junction x="27.94" y="5.08"/>
 <pinref part="R5" gate="G$1" pin="1"/>
+<wire x1="68.58" y1="5.08" x2="43.18" y2="5.08" width="0.1524" layer="91"/>
 <wire x1="43.18" y1="5.08" x2="27.94" y2="5.08" width="0.1524" layer="91"/>
 <wire x1="43.18" y1="33.02" x2="43.18" y2="5.08" width="0.1524" layer="91"/>
@@
 <pinref part="Q1" gate="G$1" pin="S"/>
 <wire x1="86.36" y1="35.56" x2="86.36" y2="5.08" width="0.1524" layer="91"/>
-<wire x1="86.36" y1="5.08" x2="68.58" y2="5.08" width="0.1524" layer="91"/>
-<junction x="68.58" y="5.08"/>
 <pinref part="C3" gate="G$1" pin="-"/>
 <wire x1="101.6" y1="20.32" x2="101.6" y2="5.08" width="0.1524" layer="91"/>
@@
 <wire x1="139.7" y1="5.08" x2="121.92" y2="5.08" width="0.1524" layer="91"/>
 <junction x="121.92" y="5.08"/>
+<pinref part="T2" gate="G$1" pin="C"/>
+<wire x1="68.58" y1="25.4" x2="68.58" y2="5.08" width="0.1524" layer="91"/>
+<junction x="68.58" y="5.08"/>
 </segment>
 <segment>
@@
 <net name="N$3" class="0">
 <segment>
+<pinref part="R6" gate="G$1" pin="2"/>
+<wire x1="58.42" y1="45.72" x2="55.88" y2="45.72" width="0.1524" layer="91"/>
+<wire x1="58.42" y1="30.48" x2="58.42" y2="45.72" width="0.1524" layer="91"/>
+<pinref part="T1" gate="G$1" pin="B"/>
+<wire x1="63.5" y1="45.72" x2="58.42" y2="45.72" width="0.1524" layer="91"/>
+<junction x="58.42" y="45.72"/>
 <pinref part="T2" gate="G$1" pin="B"/>
-<pinref part="R6" gate="G$1" pin="2"/>
-<wire x1="63.5" y1="45.72" x2="58.42" y2="45.72" width="0.1524" layer="91"/>
-<pinref part="T1" gate="G$1" pin="B"/>
-<wire x1="58.42" y1="45.72" x2="55.88" y2="45.72" width="0.1524" layer="91"/>
-<wire x1="63.5" y1="30.48" x2="58.42" y2="30.48" width="0.1524" layer="91"/>
-<wire x1="58.42" y1="30.48" x2="58.42" y2="45.72" width="0.1524" layer="91"/>
-<junction x="58.42" y="45.72"/>
+<wire x1="58.42" y1="30.48" x2="63.5" y2="30.48" width="0.1524" layer="91"/>
 </segment>
 </net>
@@
 <wire x1="-38.1" y1="45.72" x2="43.18" y2="45.72" width="0.1524" layer="91"/>
 <junction x="43.18" y="45.72"/>
-</segment>
-</net>
-<net name="N$6" class="0">
-<segment>
-<pinref part="T1" gate="G$1" pin="E"/>
-<pinref part="T2" gate="G$1" pin="C"/>
-<wire x1="68.58" y1="35.56" x2="68.58" y2="38.1" width="0.1524" layer="91"/>
-<pinref part="Q1" gate="G$1" pin="G"/>
-<wire x1="68.58" y1="38.1" x2="68.58" y2="40.64" width="0.1524" layer="91"/>
-<wire x1="81.28" y1="38.1" x2="68.58" y2="38.1" width="0.1524" layer="91"/>
-<junction x="68.58" y="38.1"/>
 </segment>
 </net>
@@
 <pinref part="U$1" gate="G$1" pin="VCC"/>
 <wire x1="15.24" y1="55.88" x2="27.94" y2="55.88" width="0.1524" layer="91"/>
-<pinref part="T2" gate="G$1" pin="E"/>
 <wire x1="27.94" y1="55.88" x2="68.58" y2="55.88" width="0.1524" layer="91"/>
-<wire x1="68.58" y1="55.88" x2="68.58" y2="50.8" width="0.1524" layer="91"/>
 <pinref part="U$1" gate="G$1" pin="DRV_COLL"/>
 <wire x1="15.24" y1="66.04" x2="27.94" y2="66.04" width="0.1524" layer="91"/>
@@
 <wire x1="-50.8" y1="68.58" x2="-50.8" y2="66.04" width="0.1524" layer="91"/>
 <junction x="-50.8" y="66.04"/>
+<pinref part="T1" gate="G$1" pin="C"/>
+<wire x1="68.58" y1="50.8" x2="68.58" y2="55.88" width="0.1524" layer="91"/>
 </segment>
 </net>
@@
 <pinref part="R11" gate="G$1" pin="1"/>
 <wire x1="330.2" y1="45.72" x2="342.9" y2="45.72" width="0.1524" layer="91"/>
+<label x="332.74" y="43.18" size="1.778" layer="95"/>
 </segment>
 </net>
@@
 <pinref part="R12" gate="G$1" pin="1"/>
 <wire x1="330.2" y1="25.4" x2="342.9" y2="25.4" width="0.1524" layer="91"/>
+<label x="332.74" y="22.86" size="1.778" layer="95"/>
 </segment>
 </net>
@@
 <pinref part="R13" gate="G$1" pin="1"/>
 <wire x1="330.2" y1="7.62" x2="342.9" y2="7.62" width="0.1524" layer="91"/>
+<label x="332.74" y="5.08" size="1.778" layer="95"/>
 </segment>
 </net>
@@
 <pinref part="R14" gate="G$1" pin="1"/>
 <wire x1="330.2" y1="-10.16" x2="342.9" y2="-10.16" width="0.1524" layer="91"/>
+<label x="332.74" y="-12.7" size="1.778" layer="95"/>
 </segment>
 </net>
@@
 <pinref part="R15" gate="G$1" pin="1"/>
 <wire x1="330.2" y1="-30.48" x2="342.9" y2="-30.48" width="0.1524" layer="91"/>
+<label x="332.74" y="-33.02" size="1.778" layer="95"/>
 </segment>
 </net>
@@
 <pinref part="R16" gate="G$1" pin="1"/>
 <wire x1="330.2" y1="-50.8" x2="342.9" y2="-50.8" width="0.1524" layer="91"/>
+<label x="332.74" y="-53.34" size="1.778" layer="95"/>
 </segment>
 </net>
@@
 <pinref part="R17" gate="G$1" pin="1"/>
 <wire x1="330.2" y1="-71.12" x2="340.36" y2="-71.12" width="0.1524" layer="91"/>
+<label x="332.74" y="-73.66" size="1.778" layer="95"/>
 </segment>
 </net>
@@
 <pinref part="R18" gate="G$1" pin="1"/>
 <wire x1="330.2" y1="-88.9" x2="340.36" y2="-88.9" width="0.1524" layer="91"/>
+<label x="332.74" y="-91.44" size="1.778" layer="95"/>
 </segment>
 </net>
@@
 <pinref part="R19" gate="G$1" pin="1"/>
 <wire x1="330.2" y1="-109.22" x2="342.9" y2="-109.22" width="0.1524" layer="91"/>
+<label x="332.74" y="-111.76" size="1.778" layer="95"/>
 </segment>
 </net>
@@
 <pinref part="R20" gate="G$1" pin="1"/>
 <wire x1="330.2" y1="-127" x2="342.9" y2="-127" width="0.1524" layer="91"/>
+<label x="332.74" y="-129.54" size="1.778" layer="95"/>
 </segment>
 </net>
@@
 <pinref part="R7" gate="G$1" pin="1"/>
 <wire x1="330.2" y1="127" x2="342.9" y2="127" width="0.1524" layer="91"/>
+<label x="332.74" y="124.46" size="1.778" layer="95"/>
 </segment>
 </net>
@@
 <pinref part="R8" gate="G$1" pin="1"/>
 <wire x1="330.2" y1="106.68" x2="340.36" y2="106.68" width="0.1524" layer="91"/>
+<label x="332.74" y="104.14" size="1.778" layer="95"/>
 </segment>
 </net>
@@
 <pinref part="R9" gate="G$1" pin="1"/>
 <wire x1="330.2" y1="86.36" x2="342.9" y2="86.36" width="0.1524" layer="91"/>
+<label x="332.74" y="83.82" size="1.778" layer="95"/>
 </segment>
 </net>
@@
 <pinref part="R10" gate="G$1" pin="1"/>
 <wire x1="330.2" y1="66.04" x2="342.9" y2="66.04" width="0.1524" layer="91"/>
+<label x="332.74" y="63.5" size="1.778" layer="95"/>
 </segment>
 </net>
@@
 </segment>
 </net>
+<net name="N$6" class="0">
+<segment>
+<pinref part="T2" gate="G$1" pin="E"/>
+<pinref part="T1" gate="G$1" pin="E"/>
+<wire x1="68.58" y1="35.56" x2="68.58" y2="38.1" width="0.1524" layer="91"/>
+<pinref part="Q1" gate="G$1" pin="G"/>
+<wire x1="68.58" y1="38.1" x2="68.58" y2="40.64" width="0.1524" layer="91"/>
+<wire x1="81.28" y1="38.1" x2="68.58" y2="38.1" width="0.1524" layer="91"/>
+<junction x="68.58" y="38.1"/>
+</segment>
+</net>

Commit message: Edit DC-DC
Parts:
- removed IC2: REG1117, burr-brown:REG1117
- added C19, C20, C21, C22: (no value), rcl:C-EUC0805K
- added C23, C25: (no value), rcl:CPOL-EUCT7343
- added C24: (no value), rcl:C-EUC0805
- added L4: SDR0604-2R2ML, SDR0604-2R2ML:SDR0604-2R2ML
- added R35, R36, R37, R38, R39, R40, R41: (no value), rcl:R-EU_R0805
- added U2: TPS562200DDCT, TPS562200DDCT:TPS562200DDCT
Connections:
- removed net N$9: C13.1, IC2.VOUT, L2.1
- new net N$61: C22.2, R36.1, U1.PB5
- new net N$65: C21.2, R37.1, U1.PB6
- new net N$66: C20.2, R38.1, U1.PB7
- new net N$67: C8.1, L2.2, U1.VDDA
- new net N$68: R41.1, U2.EN
- new net N$71: C24.1, U2.VBST
- new net N$72: C24.2, L4.1, U2.SW
- new net N$73: R39.1, R40.2, U2.VFB
- net +12V: now also C23.+, R41.2, U2.VIN; no longer IC2.VIN
- net +3V3: now also C13.1, C25.+, L2.1, L4.2, R35.2, R39.2; no longer C8.1, L2.2, U1.VDDA
- net GND: now also C19.2, C20.1, C21.1, C22.1, C23.-, C25.-, R36.2, R37.2, R38.2, R40.1, U2.GND; no longer IC2.GND, U1.PB5, U1.PB6, U1.PB7
- net N$13: now also R35.1
- net N$48: now also C19.1
Other:
- moved on the sheet: C13, C14, L2, R22, X1-1, X1-2

Commit message: Edit inductor
Parts:
- L1: value (none) -> SRR1260-221K; device rcl:L-US6000-XXX-RC -> SRR1260-221K:SRR1260-221K
Connections:
- net N$5: now also L1.2; no longer L1.1
- net N$7: now also L1.1; no longer L1.2
Changed lines of the file:
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@@
 <part name="U1" library="stm32f0" deviceset="STM32F042KXTX" device=""/>
 <part name="U$1" library="voltage_regulators" deviceset="MC34063/MC33063" device=""/>
-<part name="L1" library="rcl" library_urn="urn:adsk.eagle:library:334" deviceset="L-US" device="6000-XXX-RC" package3d_urn="urn:adsk.eagle:package:23538/1"/>
 <part name="C1" library="rcl" library_urn="urn:adsk.eagle:library:334" deviceset="CPOL-EU" device="E2.5-6" package3d_urn="urn:adsk.eagle:package:23349/1"/>
 <part name="C2" library="rcl" library_urn="urn:adsk.eagle:library:334" deviceset="C-EU" device="C0805" package3d_urn="urn:adsk.eagle:package:23617/2"/>
@@
 <part name="R40" library="rcl" library_urn="urn:adsk.eagle:library:334" deviceset="R-EU_" device="R0805" package3d_urn="urn:adsk.eagle:package:23553/2"/>
 <part name="R41" library="rcl" library_urn="urn:adsk.eagle:library:334" deviceset="R-EU_" device="R0805" package3d_urn="urn:adsk.eagle:package:23553/2"/>
+<part name="L1" library="SRR1260-221K" deviceset="SRR1260-221K" device=""/>
 </parts>
 <sheets>
@@
 <attribute name="VALUE" x="-12.7" y="71.882" size="1.778" layer="96"/>
 </instance>
-<instance part="L1" gate="G$1" x="71.12" y="60.96" smashed="yes" rot="R90">
-<attribute name="NAME" x="76.2" y="59.69" size="1.778" layer="95" rot="R180"/>
-<attribute name="VALUE" x="76.2" y="64.77" size="1.778" layer="96" rot="R180"/>
-</instance>
 <instance part="C1" gate="G$1" x="-50.8" y="33.02" smashed="yes">
 <attribute name="NAME" x="-49.657" y="33.5026" size="1.778" layer="95"/>
@@
 <attribute name="NAME" x="29.21" y="168.6814" size="1.778" layer="95" rot="R180"/>
 <attribute name="VALUE" x="29.21" y="173.482" size="1.778" layer="96" rot="R180"/>
+</instance>
+<instance part="L1" gate="G$1" x="71.12" y="60.96" smashed="yes" rot="R90">
+<attribute name="NAME" x="65.27608125" y="62.99266875" size="1.778590625" layer="95" rot="R90"/>
+<attribute name="VALUE" x="78.75321875" y="62.741090625" size="1.781090625" layer="96" rot="R90"/>
 </instance>
 </instances>
@@
 <segment>
 <pinref part="U$1" gate="G$1" pin="IPK_SENSE"/>
-<pinref part="L1" gate="G$1" pin="1"/>
 <wire x1="15.24" y1="60.96" x2="38.1" y2="60.96" width="0.1524" layer="91"/>
 <pinref part="R4" gate="G$1" pin="1"/>
@@
 <wire x1="38.1" y1="63.5" x2="38.1" y2="60.96" width="0.1524" layer="91"/>
 <junction x="38.1" y="60.96"/>
+<pinref part="L1" gate="G$1" pin="2"/>
 </segment>
 </net>
@@
 <pinref part="D1" gate="G$1" pin="A"/>
 <wire x1="86.36" y1="60.96" x2="91.44" y2="60.96" width="0.1524" layer="91"/>
-<pinref part="L1" gate="G$1" pin="2"/>
 <wire x1="78.74" y1="60.96" x2="86.36" y2="60.96" width="0.1524" layer="91"/>
 <junction x="86.36" y="60.96"/>
@@
 <wire x1="99.06" y1="73.66" x2="86.36" y2="73.66" width="0.1524" layer="91"/>
 <wire x1="86.36" y1="73.66" x2="86.36" y2="60.96" width="0.1524" layer="91"/>
+<pinref part="L1" gate="G$1" pin="1"/>
 </segment>
 </net>
