File: geiger2.sch (EAGLE design)
At the start: 109 parts, among them Q1 IRF740, Q2 CSM-7X-DU, T5 BC847, U1 STM32F042KXTX, U2 TPS562200DDCT, X1 22-23-2021, X2 22-23-2041, X3 22-23-2101, X4 22-23-2041

Commit message: Add pcb and place elements
Parts:
- added L5: (no value), dp_devices:FERRITE-0805
- C1: device rcl:CPOL-EUE2.5-6 -> rcl:CPOL-EUCT7343
- D1, D2, D3: device adafruit:SCHOTTKY-DIODEDO41-7 -> diode:DIODE-DO214AC
- Q1: value IRF740 -> IRF840; device transistor-power:IRF740 -> transistor-fet:IRF840
- T1: value (none) -> BC847BLT1SMD; device transistor:BC546-NPN-TO92-CBE -> transistor-npn:BC847BLT1SMD
- T2: device transistor:BC556A-PNP-TO92-EBC -> transistor-neu-to92:BC857C-PNP-SOT23-BEC
Connections:
- new net N$9: C14.1, C23.+, L5.1, R41.2, U2.VIN
- net +12V: now also L5.2; no longer C14.1, C23.+, R41.2, U2.VIN
Changed lines of the file:
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@@
 <setting verticaltext="up"/>
 </settings>
-<grid distance="0.1" unitdist="inch" unit="inch" style="lines" multiple="1" display="yes" altdistance="0.01" altunitdist="inch" altunit="inch"/>
+<grid distance="0.1" unitdist="inch" unit="inch" style="lines" multiple="1" display="no" altdistance="0.01" altunitdist="inch" altunit="inch"/>
 <layers>
 <layer number="1" name="Top" color="4" fill="1" visible="no" active="no"/>
@@
 <part name="U1" library="stm32f0" deviceset="STM32F042KXTX" device=""/>
 <part name="U$1" library="voltage_regulators" deviceset="MC34063/MC33063" device=""/>
-<part name="C1" library="rcl" library_urn="urn:adsk.eagle:library:334" deviceset="CPOL-EU" device="E2.5-6" package3d_urn="urn:adsk.eagle:package:23349/1"/>
+<part name="C1" library="rcl" deviceset="CPOL-EU" device="CT7343" package3d_urn="urn:adsk.eagle:package:23304/2"/>
 <part name="C2" library="rcl" library_urn="urn:adsk.eagle:library:334" deviceset="C-EU" device="C0805" package3d_urn="urn:adsk.eagle:package:23617/2"/>
-<part name="D1" library="adafruit" deviceset="SCHOTTKY-DIODE" device="DO41-7"/>
-<part name="T1" library="transistor" library_urn="urn:adsk.eagle:library:402" deviceset="*-NPN-" device="TO92-CBE" package3d_urn="urn:adsk.eagle:package:29921/2" technology="BC546"/>
-<part name="T2" library="transistor" deviceset="*-PNP-" device="TO92-EBC" technology="BC556A"/>
-<part name="Q1" library="transistor-power" library_urn="urn:adsk.eagle:library:400" deviceset="IRF740" device="" package3d_urn="urn:adsk.eagle:package:29484/3"/>
+<part name="D1" library="diode" deviceset="DIODE-" device="DO214AC" package3d_urn="urn:adsk.eagle:package:43417/2"/>
+<part name="T1" library="transistor-npn" deviceset="BC847*" device="SMD" package3d_urn="urn:adsk.eagle:package:28738/2" technology="BLT1" value="BC847BLT1SMD"/>
+<part name="T2" library="transistor-neu-to92" deviceset="*-PNP-" device="SOT23-BEC" package3d_urn="urn:adsk.eagle:package:28748/2" technology="BC857C"/>
+<part name="Q1" library="transistor-fet" deviceset="IRF840" device="" package3d_urn="urn:adsk.eagle:package:28520/1"/>
 <part name="R2" library="rcl" library_urn="urn:adsk.eagle:library:334" deviceset="R-EU_" device="R0805" package3d_urn="urn:adsk.eagle:package:23553/2"/>
 <part name="R3" library="rcl" library_urn="urn:adsk.eagle:library:334" deviceset="R-EU_" device="R0805" package3d_urn="urn:adsk.eagle:package:23553/2"/>
@@
 <part name="R6" library="rcl" library_urn="urn:adsk.eagle:library:334" deviceset="R-EU_" device="R0805" package3d_urn="urn:adsk.eagle:package:23553/2"/>
 <part name="R5" library="rcl" library_urn="urn:adsk.eagle:library:334" deviceset="R-EU_" device="R0805" package3d_urn="urn:adsk.eagle:package:23553/2"/>
-<part name="D2" library="adafruit" deviceset="SCHOTTKY-DIODE" device="DO41-7"/>
-<part name="D3" library="adafruit" deviceset="SCHOTTKY-DIODE" device="DO41-7"/>
+<part name="D2" library="diode" deviceset="DIODE-" device="DO214AC" package3d_urn="urn:adsk.eagle:package:43417/2"/>
+<part name="D3" library="diode" deviceset="DIODE-" device="DO214AC" package3d_urn="urn:adsk.eagle:package:43417/2"/>
 <part name="C5" library="rcl" deviceset="C-EU" device="C1812K"/>
 <part name="C6" library="rcl" deviceset="C-EU" device="C1812K"/>
@@
 <part name="R41" library="rcl" library_urn="urn:adsk.eagle:library:334" deviceset="R-EU_" device="R0805" package3d_urn="urn:adsk.eagle:package:23553/2"/>
 <part name="L1" library="SRR1260-221K" deviceset="SRR1260-221K" device=""/>
+<part name="L5" library="dp_devices" deviceset="FERRITE" device="-0805"/>
 </parts>
 <sheets>
@@
 <attribute name="VALUE" x="55.88" y="35.56" size="1.778" layer="96"/>
 </instance>
-<instance part="Q1" gate="G$1" x="83.82" y="40.64" smashed="yes">
-<attribute name="NAME" x="91.44" y="43.18" size="1.778" layer="95"/>
-<attribute name="VALUE" x="91.44" y="40.64" size="1.778" layer="96"/>
+<instance part="Q1" gate="G$1" x="81.28" y="40.64" smashed="yes">
+<attribute name="NAME" x="88.9" y="43.18" size="1.778" layer="95"/>
+<attribute name="VALUE" x="88.9" y="40.64" size="1.778" layer="96"/>
 </instance>
 <instance part="R2" gate="G$1" x="66.04" y="81.28" smashed="yes">
@@
 <attribute name="VALUE" x="-53.34" y="86.36" size="1.778" layer="96" rot="R90"/>
 </instance>
-<instance part="P+3" gate="1" x="17.78" y="182.88" smashed="yes">
-<attribute name="VALUE" x="15.24" y="177.8" size="1.778" layer="96" rot="R90"/>
+<instance part="P+3" gate="1" x="17.78" y="195.58" smashed="yes">
+<attribute name="VALUE" x="15.24" y="190.5" size="1.778" layer="96" rot="R90"/>
 </instance>
 <instance part="L2" gate="L" x="220.98" y="129.54" smashed="yes" rot="R90">
@@
 <attribute name="NAME" x="65.27608125" y="62.99266875" size="1.778590625" layer="95" rot="R90"/>
 <attribute name="VALUE" x="78.75321875" y="62.741090625" size="1.781090625" layer="96" rot="R90"/>
+</instance>
+<instance part="L5" gate="L" x="17.78" y="182.88" smashed="yes" rot="R180">
+<attribute name="NAME" x="15.24" y="176.53" size="1.778" layer="95" rot="R180"/>
+<attribute name="VALUE" x="15.24" y="189.23" size="1.778" layer="96" rot="R180"/>
 </instance>
 </instances>
@@
 <junction x="43.18" y="5.08"/>
 <pinref part="Q1" gate="G$1" pin="S"/>
-<wire x1="86.36" y1="35.56" x2="86.36" y2="5.08" width="0.1524" layer="91"/>
+<wire x1="86.36" y1="38.1" x2="86.36" y2="5.08" width="0.1524" layer="91"/>
 <pinref part="C3" gate="G$1" pin="-"/>
 <wire x1="101.6" y1="20.32" x2="101.6" y2="5.08" width="0.1524" layer="91"/>
@@
 <segment>
 <pinref part="Q1" gate="G$1" pin="D"/>
-<wire x1="86.36" y1="45.72" x2="86.36" y2="60.96" width="0.1524" layer="91"/>
+<wire x1="86.36" y1="43.18" x2="86.36" y2="60.96" width="0.1524" layer="91"/>
 <pinref part="D1" gate="G$1" pin="A"/>
 <wire x1="86.36" y1="60.96" x2="91.44" y2="60.96" width="0.1524" layer="91"/>
@@
 <segment>
 <pinref part="P+3" gate="1" pin="+12V"/>
-<wire x1="17.78" y1="180.34" x2="17.78" y2="170.18" width="0.1524" layer="91"/>
-<pinref part="U2" gate="G$1" pin="VIN"/>
-<wire x1="17.78" y1="170.18" x2="17.78" y2="167.64" width="0.1524" layer="91"/>
-<wire x1="17.78" y1="167.64" x2="30.48" y2="167.64" width="0.1524" layer="91"/>
-<pinref part="R41" gate="G$1" pin="2"/>
-<wire x1="30.48" y1="167.64" x2="40.64" y2="167.64" width="0.1524" layer="91"/>
-<wire x1="40.64" y1="167.64" x2="53.34" y2="167.64" width="0.1524" layer="91"/>
-<wire x1="20.32" y1="170.18" x2="17.78" y2="170.18" width="0.1524" layer="91"/>
-<junction x="17.78" y="170.18"/>
-<pinref part="C23" gate="G$1" pin="+"/>
-<wire x1="30.48" y1="165.1" x2="30.48" y2="167.64" width="0.1524" layer="91"/>
-<junction x="30.48" y="167.64"/>
-<pinref part="C14" gate="G$1" pin="1"/>
-<wire x1="40.64" y1="165.1" x2="40.64" y2="167.64" width="0.1524" layer="91"/>
-<junction x="40.64" y="167.64"/>
+<wire x1="17.78" y1="193.04" x2="17.78" y2="190.5" width="0.1524" layer="91"/>
+<pinref part="L5" gate="L" pin="2"/>
 </segment>
 </net>
@@
 <pinref part="Q1" gate="G$1" pin="G"/>
 <wire x1="68.58" y1="38.1" x2="68.58" y2="40.64" width="0.1524" layer="91"/>
-<wire x1="81.28" y1="38.1" x2="68.58" y2="38.1" width="0.1524" layer="91"/>
+<wire x1="76.2" y1="38.1" x2="68.58" y2="38.1" width="0.1524" layer="91"/>
 <junction x="68.58" y="38.1"/>
 </segment>
@@
 </segment>
 </net>
+<net name="N$9" class="0">
+<segment>
+<pinref part="U2" gate="G$1" pin="VIN"/>
+<wire x1="17.78" y1="170.18" x2="17.78" y2="167.64" width="0.1524" layer="91"/>
+<wire x1="17.78" y1="167.64" x2="30.48" y2="167.64" width="0.1524" layer="91"/>
+<pinref part="R41" gate="G$1" pin="2"/>
+<wire x1="30.48" y1="167.64" x2="40.64" y2="167.64" width="0.1524" layer="91"/>
+<wire x1="40.64" y1="167.64" x2="53.34" y2="167.64" width="0.1524" layer="91"/>
+<wire x1="20.32" y1="170.18" x2="17.78" y2="170.18" width="0.1524" layer="91"/>
+<junction x="17.78" y="170.18"/>
+<pinref part="C23" gate="G$1" pin="+"/>
+<wire x1="30.48" y1="165.1" x2="30.48" y2="167.64" width="0.1524" layer="91"/>
+<junction x="30.48" y="167.64"/>
+<pinref part="C14" gate="G$1" pin="1"/>
+<wire x1="40.64" y1="165.1" x2="40.64" y2="167.64" width="0.1524" layer="91"/>
+<junction x="40.64" y="167.64"/>
+<wire x1="17.78" y1="175.26" x2="17.78" y2="170.18" width="0.1524" layer="91"/>
+<pinref part="L5" gate="L" pin="1"/>
+</segment>
+</net>

Commit message: Edit board
Parts:
- T1: value BC847BLT1SMD -> BC847
- U$1: value MC34063/MC33063 -> MC34063
Changed lines of the file:
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@@
 <?xml version="1.0" encoding="utf-8"?>
 <!DOCTYPE eagle SYSTEM "eagle.dtd">
-<eagle version="9.4.1">
+<eagle version="9.3.0">
 <drawing>
 <settings>
@@
 <parts>
 <part name="U1" library="stm32f0" deviceset="STM32F042KXTX" device=""/>
-<part name="U$1" library="voltage_regulators" deviceset="MC34063/MC33063" device=""/>
+<part name="U$1" library="voltage_regulators" deviceset="MC34063/MC33063" device="" value="MC34063"/>
 <part name="C1" library="rcl" deviceset="CPOL-EU" device="CT7343" package3d_urn="urn:adsk.eagle:package:23304/2"/>
 <part name="C2" library="rcl" library_urn="urn:adsk.eagle:library:334" deviceset="C-EU" device="C0805" package3d_urn="urn:adsk.eagle:package:23617/2"/>
 <part name="D1" library="diode" deviceset="DIODE-" device="DO214AC" package3d_urn="urn:adsk.eagle:package:43417/2"/>
-<part name="T1" library="transistor-npn" deviceset="BC847*" device="SMD" package3d_urn="urn:adsk.eagle:package:28738/2" technology="BLT1" value="BC847BLT1SMD"/>
+<part name="T1" library="transistor-npn" deviceset="BC847*" device="SMD" package3d_urn="urn:adsk.eagle:package:28738/2" technology="BLT1" value="BC847"/>
 <part name="T2" library="transistor-neu-to92" deviceset="*-PNP-" device="SOT23-BEC" package3d_urn="urn:adsk.eagle:package:28748/2" technology="BC857C"/>
 <part name="Q1" library="transistor-fet" deviceset="IRF840" device="" package3d_urn="urn:adsk.eagle:package:28520/1"/>

Commit message: Add routing
Parts:
- removed C11: (no value), rcl:C-EUC0805
Connections:
- removed net N$38: OK5.EMIT
- net +3V3: no longer C11.1
- net GND: now also OK5.EMIT; no longer C11.2
Changed lines of the file:
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@@
 <?xml version="1.0" encoding="utf-8"?>
 <!DOCTYPE eagle SYSTEM "eagle.dtd">
-<eagle version="9.3.0">
+<eagle version="9.4.1">
 <drawing>
 <settings>
@@
 <part name="GND3" library="supply1" library_urn="urn:adsk.eagle:library:371" deviceset="GND" device=""/>
 <part name="C10" library="rcl" library_urn="urn:adsk.eagle:library:334" deviceset="C-EU" device="C0805" package3d_urn="urn:adsk.eagle:package:23617/2"/>
-<part name="C11" library="rcl" library_urn="urn:adsk.eagle:library:334" deviceset="C-EU" device="C0805" package3d_urn="urn:adsk.eagle:package:23617/2"/>
 <part name="+3V1" library="supply1" library_urn="urn:adsk.eagle:library:371" deviceset="+3V3" device=""/>
 <part name="C12" library="rcl" library_urn="urn:adsk.eagle:library:334" deviceset="C-EU" device="C0805" package3d_urn="urn:adsk.eagle:package:23617/2"/>
@@
 <attribute name="VALUE" x="174.244" y="114.681" size="1.778" layer="96"/>
 </instance>
-<instance part="C11" gate="G$1" x="185.42" y="114.3" smashed="yes">
-<attribute name="NAME" x="186.944" y="114.681" size="1.778" layer="95"/>
-<attribute name="VALUE" x="186.944" y="109.601" size="1.778" layer="96"/>
-</instance>
 <instance part="+3V1" gate="G$1" x="172.72" y="137.16" smashed="yes">
 <attribute name="VALUE" x="170.18" y="132.08" size="1.778" layer="96" rot="R90"/>
@@
 <attribute name="VALUE" x="386.842" y="133.35" size="1.778" layer="96" rot="R90"/>
 </instance>
-<instance part="GND22" gate="1" x="381" y="35.56" smashed="yes">
-<attribute name="VALUE" x="378.46" y="33.02" size="1.778" layer="96"/>
+<instance part="GND22" gate="1" x="381" y="38.1" smashed="yes">
+<attribute name="VALUE" x="378.46" y="35.56" size="1.778" layer="96"/>
 </instance>
 <instance part="GND23" gate="1" x="381" y="15.24" smashed="yes">
@@
 <wire x1="198.12" y1="96.52" x2="187.96" y2="96.52" width="0.1524" layer="91"/>
 <wire x1="187.96" y1="96.52" x2="187.96" y2="93.98" width="0.1524" layer="91"/>
-<pinref part="C11" gate="G$1" pin="2"/>
-<wire x1="185.42" y1="109.22" x2="185.42" y2="96.52" width="0.1524" layer="91"/>
-<wire x1="185.42" y1="96.52" x2="187.96" y2="96.52" width="0.1524" layer="91"/>
 <junction x="187.96" y="96.52"/>
 <pinref part="C8" gate="G$1" pin="2"/>
@@
 <pinref part="C10" gate="G$1" pin="2"/>
 <wire x1="172.72" y1="114.3" x2="172.72" y2="96.52" width="0.1524" layer="91"/>
-<wire x1="172.72" y1="96.52" x2="185.42" y2="96.52" width="0.1524" layer="91"/>
-<junction x="185.42" y="96.52"/>
+<wire x1="172.72" y1="96.52" x2="187.96" y2="96.52" width="0.1524" layer="91"/>
 </segment>
 <segment>
@@
 <junction x="134.62" y="137.16"/>
 </segment>
+<segment>
+<pinref part="OK5" gate="A" pin="EMIT"/>
+<wire x1="381" y1="40.64" x2="375.92" y2="40.64" width="0.1524" layer="91"/>
+<pinref part="GND22" gate="1" pin="GND"/>
+</segment>
 </net>
 <net name="N$3" class="0">
@@
 <pinref part="U1" gate="G$1" pin="VDD"/>
 <wire x1="236.22" y1="109.22" x2="236.22" y2="124.46" width="0.1524" layer="91"/>
-<wire x1="226.06" y1="106.68" x2="226.06" y2="119.38" width="0.1524" layer="91"/>
+<wire x1="226.06" y1="106.68" x2="226.06" y2="124.46" width="0.1524" layer="91"/>
 <junction x="226.06" y="124.46"/>
-<wire x1="226.06" y1="119.38" x2="226.06" y2="124.46" width="0.1524" layer="91"/>
 <pinref part="C9" gate="G$1" pin="1"/>
 <wire x1="210.82" y1="106.68" x2="210.82" y2="109.22" width="0.1524" layer="91"/>
 <wire x1="210.82" y1="109.22" x2="236.22" y2="109.22" width="0.1524" layer="91"/>
 <junction x="236.22" y="109.22"/>
-<pinref part="C11" gate="G$1" pin="1"/>
-<wire x1="185.42" y1="116.84" x2="185.42" y2="119.38" width="0.1524" layer="91"/>
-<wire x1="185.42" y1="119.38" x2="226.06" y2="119.38" width="0.1524" layer="91"/>
-<junction x="226.06" y="119.38"/>
 <pinref part="L2" gate="L" pin="1"/>
 <wire x1="213.36" y1="129.54" x2="172.72" y2="129.54" width="0.1524" layer="91"/>
@@
 </segment>
 </net>
-<net name="N$38" class="0">
-<segment>
-<pinref part="OK5" gate="A" pin="EMIT"/>
-<wire x1="375.92" y1="40.64" x2="378.46" y2="40.64" width="0.1524" layer="91"/>
-<pinref part="GND22" gate="1" pin="GND"/>
-<wire x1="381" y1="38.1" x2="381" y2="40.64" width="0.1524" layer="91"/>
-<wire x1="381" y1="40.64" x2="378.46" y2="40.64" width="0.1524" layer="91"/>
-</segment>
-</net>
