File: geiger2.brd (EAGLE design)
At the start: 160 x 100 mm, 110 parts, among them Q1 IRF840, Q2 CSM-7X-DU, T1 BC847BLT1SMD, T5 BC847, U1 STM32F042KXTX, U2 TPS562200DDCT, X1 22-23-2021, X2 22-23-2041, X3 22-23-2101, X4 22-23-2041

Commit message: Edit board
Parts:
- T1: value BC847BLT1SMD -> BC847
- U$1: value MC34063/MC33063 -> MC34063
- moved X3 65.6 mm to (139.7, 2.54), flipped to the bottom, turned to 180 degrees
- moved X2 41.8 mm to (152.4, 30.5), flipped to the bottom
- moved JP3 40.9 mm to (149.9, 39.4), flipped to the bottom, turned to 0 degrees
- moved JP1 38.6 mm to (141.0, 39.4), flipped to the bottom, turned to 180 degrees
- moved D4 38.4 mm to (143.5, 14.0), turned to 90 degrees
- moved SG1 38.2 mm to (151.1, 17.8)
- moved R6 36.9 mm to (17.8, 12.7), turned to 270 degrees
- moved T2 36.6 mm to (21.6, 12.7)
- moved R1 34.7 mm to (7.62, 22.9), turned to 180 degrees
- moved R5 34.3 mm to (17.8, 19.1), turned to 270 degrees
- moved R2 32.1 mm to (55.9, 24.1)
- moved T5 30.5 mm to (143.5, 20.3), turned to 180 degrees
- moved C2 30.2 mm to (14.0, 22.9), turned to 180 degrees
- moved T1 30.2 mm to (21.6, 17.8), turned to 0 degrees
- moved X4 30.2 mm to (43.2, 0.00), flipped to the bottom, turned to 180 degrees
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
Commit message: Add routing
Parts:
- removed C11: (no value), rcl:C0805
- moved X3 57.5 mm to (82.5, 8.64), turned to 0 degrees
- moved R20 55.4 mm to (65.5, 9.14)
- moved OK14 55.0 mm to (66.0, 8.89)
- moved OK13 53.7 mm to (59.7, 8.89)
- moved R19 53.7 mm to (59.7, 9.91)
- moved R18 52.7 mm to (53.1, 9.91)
- moved OK12 52.5 mm to (53.3, 8.89)
- moved R17 51.4 mm to (46.7, 9.65)
- moved OK11 51.2 mm to (47.0, 8.89)
- moved OK10 49.9 mm to (40.6, 8.89)
- moved R16 49.9 mm to (40.6, 9.91)
- moved OK5 47.4 mm to (99.1, 8.89)
- moved R12 46.3 mm to (105.7, 9.40), turned to 0 degrees
- moved OK6 46.2 mm to (105.4, 8.89)
- moved R11 46.1 mm to (97.8, 9.65), turned to 0 degrees
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Connections:
- removed net N$38: OK5.3
- net +3V3: no longer C11.1
- net GND: now also OK5.3; no longer C11.2
Routing:
- net GND: track 0.00 -> 585.9 mm, vias 0 -> 7
- net +3V3: track 0.00 -> 194.6 mm, vias 0 -> 11
- net OK13: track 0.00 -> 123.7 mm, vias 0 -> 4
- net OK11: track 0.00 -> 104.3 mm, vias 0 -> 2
- net OK12: track 0.00 -> 100.0 mm, vias 0 -> 4
- net OK14: track 0.00 -> 93.2 mm, vias 0 -> 4
- net N$66: track 0.00 -> 91.7 mm, vias 0 -> 3
- net OK6: track 0.00 -> 61.0 mm, vias 0 -> 2
- net N$61: track 0.00 -> 57.9 mm, vias 0 -> 2
- net N$42: track 0.00 -> 51.9 mm, vias 0 -> 1
- net N$41: track 0.00 -> 49.0 mm, vias 0 -> 1
- net OK7: track 0.00 -> 47.2 mm, vias 0 -> 2
- net N$5: track 0.00 -> 43.9 mm, vias 0 -> 1
- net N$55: track 0.00 -> 43.1 mm, vias 0 -> 3
- net OK8: track 0.00 -> 42.6 mm, vias 0 -> 2
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Other:
- board size 160 x 100 mm -> 128.2 x 44.1 mm

Commit message: edit board
Parts:
- moved R41 26.5 mm to (67.6, 29.7), turned to 180 degrees
- moved R23 19.3 mm to (62.5, 19.6), turned to 270 degrees
- moved R24 18.7 mm to (65.5, 19.6), turned to 90 degrees
- moved R27 11.8 mm to (79.0, 20.3), turned to 180 degrees
- moved T3 11.2 mm to (74.7, 20.3)
- moved R25 8.92 mm to (72.6, 23.9)
- moved R26 8.65 mm to (73.7, 27.4), turned to 90 degrees
- moved L5 8.13 mm to (48.8, 36.8)
- moved C23 8.03 mm to (61.2, 35.6)
- moved C24 7.40 mm to (66.0, 38.1)
- moved L4 7.27 mm to (53.8, 35.3), turned to 0 degrees
- moved C17 6.94 mm to (65.3, 24.1)
- moved U2 6.84 mm to (66.0, 34.0)
- moved D1 6.35 mm to (34.3, 17.0)
- moved R28 6.14 mm to (74.2, 16.3)
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Routing:
- net +3V3: track 194.6 -> 109.5 mm, vias 11 -> 7
- net GND: track 585.9 -> 514.2 mm, vias 7 -> 4
- net OK13: track 123.7 -> 84.2 mm, vias 4 -> 3
- net N$5: track 43.9 -> 14.7 mm
- net +12V: track 39.1 -> 15.7 mm
- net N$68: track 23.6 -> 5.96 mm
- net OK12: track 100.0 -> 108.4 mm, vias 4 -> 2
- net N$9: track 29.7 -> 23.9 mm, vias 1 -> 0
- net N$7: track 42.5 -> 37.0 mm
- net N$57: track 39.6 -> 34.5 mm
- net N$73: track 14.8 -> 19.1 mm, vias 0 -> 2
- net N$53: track 8.46 -> 5.25 mm
- net N$2: track 23.9 -> 27.0 mm
- net N$54: track 11.6 -> 8.62 mm
- net OK11: track 104.3 -> 107.3 mm
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